File: sbus-to-ztex/sbus-to-ztex.sch (KiCad schematic (older format))
At the start: 0 parts

Commit message: thinking about a V1.3
Changed lines of the file:
@@
 EESchema Schematic File Version 4
-LIBS:sbus-to-ztex-cache
-EELAYER 26 0
+EELAYER 30 0
 EELAYER END
 $Descr A4 11693 8268
 encoding utf-8
-Sheet 1 6
+Sheet 1 9
 Title "sbus-to-ztex root"
 Date ""
@@
 F1 "usb.sch" 50
 $EndSheet
+$Sheet
+S 2400 2700 1200 550
+U 652243BA
+F0 "hdmi" 50
+F1 "hdmi.sch" 50
+$EndSheet
+$Sheet
+S 900  3475 1200 525
+U 6530AC84
+F0 "i2c" 50
+F1 "i2c.sch" 50
+$EndSheet
+$Sheet
+S 2400 3475 1200 525
+U 65374E5B
+F0 "clock" 50
+F1 "clock.sch" 50
+$EndSheet
 $EndSCHEMATC

Commit message: more V1.3
Parts:
- added GRAPHIC1: LogoLitex, For_SeeedStudio:litex_logo, symbol logo:LogoLitex
- added GRAPHIC2: LogoNetBSD, For_SeeedStudio:netbsd_logo, symbol logo:LogoNetBSD
Changed lines of the file:
@@
-$EndSheet
-$Sheet
-S 900  1800 1200 600
-U 5F69F4EF
-F0 "sdcard.sch" 50
-F1 "sdcard.sch" 50
 $EndSheet
 $Sheet
@@
 F1 "clock.sch" 50
 $EndSheet
+$Sheet
+S 900  1800 1200 600
+U 65499504
+F0 "pmod" 50
+F1 "pmod.sch" 50
+$EndSheet
+$Comp
+L logo:LogoLitex GRAPHIC1
+U 1 1 654C91E8
+P 4250 1275
+F 0 "GRAPHIC1" H 4478 1271 50  0000 L CNN
+F 1 "LogoLitex" H 4478 1180 50  0000 L CNN
+F 2 "For_SeeedStudio:litex_logo" H 4250 1275 50  0001 C CNN
+F 3 "" H 4250 1275 50  0001 C CNN
+F 4 "DNP" H 4250 1275 50  0001 C CNN "DNP"
+	1    4250 1275
+	1    0    0    -1
+$EndComp
+$Comp
+L logo:LogoNetBSD GRAPHIC2
+U 1 1 654C967D
+P 4300 1625
+F 0 "GRAPHIC2" H 4578 1721 50  0000 L CNN
+F 1 "LogoNetBSD" H 4578 1630 50  0000 L CNN
+F 2 "For_SeeedStudio:netbsd_logo" H 4300 1625 50  0001 C CNN
+F 3 "" H 4300 1625 50  0001 C CNN
+F 4 "DNP" H 4300 1625 50  0001 C CNN "DNP"
+	1    4300 1625
+	1    0    0    -1
+$EndComp
 $EndSCHEMATC
