File: sbus-to-ztex/sbus.sch (KiCad schematic (older format))
At the start: 23 parts, among them U1 SN74CB3T16211DGGR, U2 SN74CB3T16211DGGR, U3 SN74CB3T16211DGGR, U4 SN74CB3T3125PW

Commit message: thinking about a V1.3
Parts:
- removed C8: 100nF, Capacitor_SMD:C_0603_1608Metric, symbol Device:C
- removed U4: SN74CB3T3125PW, Package_SO:TSSOP-14_4.4x5mm_P0.65mm, symbol ul_SN74CB3T3125PW:SN74CB3T3125PW
- added C27: 100nF 0402, Capacitor_SMD:C_0402_1005Metric, symbol Device:C
- added U10, U4: 74CB3T1G125, Package_TO_SOT_SMD:SOT-23-5, symbol 74xGxx:74CB3T1G125
- C10, C11, C13, C31, C4, C7: value 100nF -> 100nF 0402; footprint Capacitor_SMD:C_0603_1608Metric -> Capacitor_SMD:C_0402_1005Metric; LCSC ? -> (none); MNF1_URL www.yageo.com -> (none); MPN CC0603KRX7R8BB104 -> CL05B104KO5NNNC; Mouser 603-CC603KRX7R8BB104 -> (none)
- C12: value 100nF -> 100nF 0402; footprint Capacitor_SMD:C_0603_1608Metric -> Capacitor_SMD:C_0402_1005Metric; LCSC ? -> (none); MNF1_URL www.yageo.com -> (none); MPN CC0603KRX7R8BB104 -> CL05B104KO5NNNC; Mouser 603-CC60KRX7R8BB104 -> (none)
- R1, R13, R2, R30, R31, R5, R6: footprint Resistor_SMD:R_0603_1608Metric -> Resistor_SMD:R_0402_1005Metric; MPN 0603WAF1002T5E -> 0402WGF1002TCE
- U_INT1, U_INT2, U_INT3: footprint Package_TO_SOT_SMD:SOT-23-6 -> For_SeeedStudio:SOT65P210X110-6N; MPN SN74LVC2G07DBVR -> SN74LVC2G07DCKR
- U_INT1, U_INT2, U_INT3: footprint (none) -> For_SeeedStudio:SOT65P210X110-6N; MPN (none) -> SN74LVC2G07DCKR
Connections:
- net +3V3: now also C27.1, U10.5 (VCC), U4.5 (VCC)
- net GND: now also C27.2, U10.3 (GND), U4.3 (GND)
- net SBUS_3V3_ACK[0]*: now also U1.24 (2A8); no longer U1.51 (1B4)
- net SBUS_3V3_ACK[1]*: now also U1.15 (2A1); no longer U1.46 (1B8)
- net SBUS_3V3_ACK[2]*: now also U1.7 (1A6); no longer U1.42 (1B12)
- net SBUS_3V3_AS*: now also U3.27 (2A11); no longer U3.52 (1B3)
- net SBUS_3V3_BG*: now also U10.4 (B)
- net SBUS_3V3_BR*: now also U4.4 (B)
- net SBUS_3V3_CLK: now also U3.28 (2A12); no longer U3.51 (1B4)
- net SBUS_3V3_D[00]: now also U3.25 (2A9); no longer U3.48 (1B6)
- net SBUS_3V3_D[01]: now also U3.24 (2A8); no longer U3.50 (1B5)
- net SBUS_3V3_D[02]: now also U3.23 (2A7); no longer U3.46 (1B8)
- net SBUS_3V3_D[03]: now also U3.22 (2A6); no longer U3.47 (1B7)
- net SBUS_3V3_D[04]: now also U3.21 (2A5); no longer U3.44 (1B10)
- net SBUS_3V3_D[05]: now also U3.20 (2A4); no longer U3.45 (1B9)
- net SBUS_3V3_D[06]: now also U3.18 (2A3); no longer U3.43 (1B11)
- net SBUS_3V3_D[07]: now also U3.16 (2A2); no longer U3.42 (1B12)
- net SBUS_3V3_D[08]: now also U3.15 (2A1); no longer U3.41 (2B1)
- net SBUS_3V3_D[09]: now also U3.14 (1A12); no longer U3.40 (2B2)
- net SBUS_3V3_D[10]: now also U3.13 (1A11); no longer U3.39 (2B3)
- net SBUS_3V3_D[11]: now also U3.12 (1A10); no longer U3.37 (2B4)
- net SBUS_3V3_D[12]: now also U3.11 (1A9); no longer U3.36 (2B5)
- net SBUS_3V3_D[13]: now also U3.10 (1A8); no longer U3.35 (2B6)
- net SBUS_3V3_D[14]: now also U3.9 (1A7); no longer U3.34 (2B7)
- net SBUS_3V3_D[15]: now also U3.7 (1A6); no longer U3.33 (2B8)
- net SBUS_3V3_D[16]: now also U3.6 (1A5); no longer U3.32 (2B9)
- net SBUS_3V3_D[17]: now also U3.5 (1A4); no longer U3.31 (2B10)
- net SBUS_3V3_D[18]: now also U3.4 (1A3); no longer U3.30 (2B11)
- net SBUS_3V3_D[19]: now also U3.3 (1A2); no longer U3.29 (2B12)
- net SBUS_3V3_D[20]: now also U3.2 (1A1); no longer U2.54 (1B1)
- net SBUS_3V3_D[21]: now also U2.28 (2A12); no longer U2.53 (1B2)
- net SBUS_3V3_D[22]: now also U2.27 (2A11); no longer U2.52 (1B3)
- net SBUS_3V3_D[23]: now also U2.26 (2A10); no longer U2.51 (1B4)
- net SBUS_3V3_D[24]: now also U2.25 (2A9); no longer U2.50 (1B5)
- net SBUS_3V3_D[25]: now also U2.24 (2A8); no longer U2.48 (1B6)
- net SBUS_3V3_D[26]: now also U2.23 (2A7); no longer U2.47 (1B7)
- net SBUS_3V3_D[27]: now also U2.22 (2A6); no longer U2.46 (1B8)
- net SBUS_3V3_D[28]: now also U2.21 (2A5); no longer U2.45 (1B9)
- net SBUS_3V3_D[29]: now also U2.20 (2A4); no longer U2.44 (1B10)
- net SBUS_3V3_D[30]: now also U2.18 (2A3); no longer U2.43 (1B11)
- net SBUS_3V3_D[31]: now also U2.16 (2A2); no longer U2.42 (1B12)
- net SBUS_3V3_EER*: now also U2.4 (1A3); no longer U1.54 (1B1)
- net SBUS_3V3_INT[3]*: now also R31.2, U_INT1.3; no longer R30.2, U_INT1.1
- net SBUS_3V3_INT[4]*: now also R30.2, U_INT1.1; no longer R31.2, U_INT1.3
- net SBUS_3V3_PA[00]: now also U2.10 (1A8); no longer U2.36 (2B5)
- net SBUS_3V3_PA[01]: now also U2.11 (1A9); no longer U2.35 (2B6)
- net SBUS_3V3_PA[02]: now also U2.7 (1A6); no longer U2.34 (2B7)
- net SBUS_3V3_PA[03]: now also U2.9 (1A7); no longer U2.33 (2B8)
- net SBUS_3V3_PA[04]: now also U2.5 (1A4); no longer U2.32 (2B9)
- net SBUS_3V3_PA[05]: now also U2.6 (1A5); no longer U2.31 (2B10)
- net SBUS_3V3_PA[06]: now also U2.2 (1A1); no longer U2.30 (2B11)
- net SBUS_3V3_PA[07]: now also U2.3 (1A2); no longer U2.29 (2B12)
- net SBUS_3V3_PA[08]: now also U1.27 (2A11); no longer U1.53 (1B2)
- net SBUS_3V3_PA[09]: now also U1.28 (2A12); no longer U1.52 (1B3)
- net SBUS_3V3_PA[10]: now also U1.25 (2A9); no longer U1.50 (1B5)
- net SBUS_3V3_PA[11]: now also U1.26 (2A10); no longer U1.48 (1B6)
- net SBUS_3V3_PA[12]: now also U1.22 (2A6); no longer U1.47 (1B7)
- net SBUS_3V3_PA[13]: now also U1.23 (2A7); no longer U1.45 (1B9)
- net SBUS_3V3_PA[14]: now also U1.20 (2A4); no longer U1.44 (1B10)
- net SBUS_3V3_PA[15]: now also U1.21 (2A5); no longer U1.43 (1B11)
- net SBUS_3V3_PA[16]: now also U1.16 (2A2); no longer U1.41 (2B1)
- net SBUS_3V3_PA[17]: now also U1.18 (2A3); no longer U1.40 (2B2)
- net SBUS_3V3_PA[18]: now also U1.13 (1A11); no longer U1.39 (2B3)
- net SBUS_3V3_PA[19]: now also U1.14 (1A12); no longer U1.37 (2B4)
- net SBUS_3V3_PA[20]: now also U1.11 (1A9); no longer U1.36 (2B5)
- net SBUS_3V3_PA[21]: now also U1.12 (1A10); no longer U1.35 (2B6)
- net SBUS_3V3_PA[22]: now also U1.9 (1A7); no longer U1.34 (2B7)
- net SBUS_3V3_PA[23]: now also U1.10 (1A8); no longer U1.33 (2B8)
- net SBUS_3V3_PA[24]: now also U1.5 (1A4); no longer U1.32 (2B9)
- net SBUS_3V3_PA[25]: now also U1.6 (1A5); no longer U1.31 (2B10)
- net SBUS_3V3_PA[26]: now also U1.3 (1A2); no longer U1.29 (2B12)
- net SBUS_3V3_PA[27]: now also U1.4 (1A3); no longer U1.30 (2B11)
- net SBUS_3V3_PPRD: now also U2.13 (1A11); no longer U2.37 (2B4)
- net SBUS_3V3_RST*: now also U1.2 (1A1); no longer U3.54 (1B1)
- net SBUS_3V3_SEL*: now also U3.26 (2A10); no longer U3.53 (1B2)
- net SBUS_3V3_SIZ[0]: now also U2.14 (1A12); no longer U2.41 (2B1)
- net SBUS_3V3_SIZ[1]: now also U2.15 (2A1); no longer U2.40 (2B2)
- net SBUS_3V3_SIZ[2]: now also U2.12 (1A10); no longer U2.39 (2B3)
- net SBUS_5V_ACK[0]*: now also U1.33 (2B8); no longer U1.5 (1A4)
- net SBUS_5V_ACK[1]*: now also U1.41 (2B1); no longer U1.10 (1A8)
- net SBUS_5V_ACK[2]*: now also U1.48 (1B6); no longer U1.14 (1A12)
- net SBUS_5V_AS*: now also U3.30 (2B11); no longer U3.4 (1A3)
- net SBUS_5V_BG*: now also U10.2 (A)
- net SBUS_5V_BR*: now also U4.2 (A)
- net SBUS_5V_CLK: now also U3.29 (2B12); no longer U3.5 (1A4)
- net SBUS_5V_D[00]: now also U3.32 (2B9); no longer U3.7 (1A6)
- net SBUS_5V_D[01]: now also U3.33 (2B8); no longer U3.6 (1A5)
- net SBUS_5V_D[02]: now also U3.34 (2B7); no longer U3.10 (1A8)
- net SBUS_5V_D[03]: now also U3.35 (2B6); no longer U3.9 (1A7)
- net SBUS_5V_D[04]: now also U3.36 (2B5); no longer U3.12 (1A10)
- net SBUS_5V_D[05]: now also U3.37 (2B4); no longer U3.11 (1A9)
- net SBUS_5V_D[06]: now also U3.39 (2B3); no longer U3.13 (1A11)
- net SBUS_5V_D[07]: now also U3.40 (2B2); no longer U3.14 (1A12)
- net SBUS_5V_D[08]: now also U3.41 (2B1); no longer U3.15 (2A1)
- net SBUS_5V_D[09]: now also U3.42 (1B12); no longer U3.16 (2A2)
- net SBUS_5V_D[10]: now also U3.43 (1B11); no longer U3.18 (2A3)
- net SBUS_5V_D[11]: now also U3.44 (1B10); no longer U3.20 (2A4)
- net SBUS_5V_D[12]: now also U3.45 (1B9); no longer U3.21 (2A5)
- net SBUS_5V_D[13]: now also U3.46 (1B8); no longer U3.22 (2A6)
- net SBUS_5V_D[14]: now also U3.47 (1B7); no longer U3.23 (2A7)
- net SBUS_5V_D[15]: now also U3.48 (1B6); no longer U3.24 (2A8)
- net SBUS_5V_D[16]: now also U3.50 (1B5); no longer U3.25 (2A9)
- net SBUS_5V_D[17]: now also U3.51 (1B4); no longer U3.26 (2A10)
- net SBUS_5V_D[18]: now also U3.52 (1B3); no longer U3.27 (2A11)
- net SBUS_5V_D[19]: now also U3.53 (1B2); no longer U3.28 (2A12)
- net SBUS_5V_D[20]: now also U3.54 (1B1); no longer U2.2 (1A1)
- net SBUS_5V_D[21]: now also U2.29 (2B12); no longer U2.3 (1A2)
- net SBUS_5V_D[22]: now also U2.30 (2B11); no longer U2.4 (1A3)
- net SBUS_5V_D[23]: now also U2.31 (2B10); no longer U2.5 (1A4)
- net SBUS_5V_D[24]: now also U2.32 (2B9); no longer U2.6 (1A5)
- net SBUS_5V_D[25]: now also U2.33 (2B8); no longer U2.7 (1A6)
- net SBUS_5V_D[26]: now also U2.34 (2B7); no longer U2.9 (1A7)
- net SBUS_5V_D[27]: now also U2.35 (2B6); no longer U2.10 (1A8)
- net SBUS_5V_D[28]: now also U2.36 (2B5); no longer U2.11 (1A9)
- net SBUS_5V_D[29]: now also U2.37 (2B4); no longer U2.12 (1A10)
- net SBUS_5V_D[30]: now also U2.39 (2B3); no longer U2.13 (1A11)
- net SBUS_5V_D[31]: now also U2.40 (2B2); no longer U2.14 (1A12)
- net SBUS_5V_EER*: now also U2.52 (1B3); no longer U1.2 (1A1)
- net SBUS_5V_INT[3]*: now also U_INT1.4; no longer U_INT1.6
- net SBUS_5V_INT[4]*: now also U_INT1.6; no longer U_INT1.4
- net SBUS_5V_PA[00]: now also U2.46 (1B8); no longer U2.21 (2A5)
- net SBUS_5V_PA[01]: now also U2.45 (1B9); no longer U2.22 (2A6)
- net SBUS_5V_PA[02]: now also U2.48 (1B6); no longer U2.23 (2A7)
- net SBUS_5V_PA[03]: now also U2.47 (1B7); no longer U2.24 (2A8)
- net SBUS_5V_PA[04]: now also U2.51 (1B4); no longer U2.25 (2A9)
- net SBUS_5V_PA[05]: now also U2.50 (1B5); no longer U2.26 (2A10)
- net SBUS_5V_PA[06]: now also U2.54 (1B1); no longer U2.27 (2A11)
- net SBUS_5V_PA[07]: now also U2.53 (1B2); no longer U2.28 (2A12)
- net SBUS_5V_PA[08]: now also U1.30 (2B11); no longer U1.3 (1A2)
- net SBUS_5V_PA[09]: now also U1.29 (2B12); no longer U1.4 (1A3)
- net SBUS_5V_PA[10]: now also U1.32 (2B9); no longer U1.6 (1A5)
- net SBUS_5V_PA[11]: now also U1.31 (2B10); no longer U1.7 (1A6)
- net SBUS_5V_PA[12]: now also U1.35 (2B6); no longer U1.9 (1A7)
- net SBUS_5V_PA[13]: now also U1.34 (2B7); no longer U1.11 (1A9)
- net SBUS_5V_PA[14]: now also U1.37 (2B4); no longer U1.12 (1A10)
- net SBUS_5V_PA[15]: now also U1.36 (2B5); no longer U1.13 (1A11)
- net SBUS_5V_PA[16]: now also U1.40 (2B2); no longer U1.15 (2A1)
- net SBUS_5V_PA[17]: now also U1.39 (2B3); no longer U1.16 (2A2)
- net SBUS_5V_PA[18]: now also U1.43 (1B11); no longer U1.18 (2A3)
- net SBUS_5V_PA[19]: now also U1.42 (1B12); no longer U1.20 (2A4)
- net SBUS_5V_PA[20]: now also U1.45 (1B9); no longer U1.21 (2A5)
- net SBUS_5V_PA[21]: now also U1.44 (1B10); no longer U1.22 (2A6)
- net SBUS_5V_PA[22]: now also U1.47 (1B7); no longer U1.23 (2A7)
- net SBUS_5V_PA[23]: now also U1.46 (1B8); no longer U1.24 (2A8)
- net SBUS_5V_PA[24]: now also U1.51 (1B4); no longer U1.25 (2A9)
- net SBUS_5V_PA[25]: now also U1.50 (1B5); no longer U1.26 (2A10)
- net SBUS_5V_PA[26]: now also U1.53 (1B2); no longer U1.28 (2A12)
- net SBUS_5V_PA[27]: now also U1.52 (1B3); no longer U1.27 (2A11)
- net SBUS_5V_PPRD: now also U2.43 (1B11); no longer U2.20 (2A4)
- net SBUS_5V_RST*: now also U1.54 (1B1); no longer U3.2 (1A1)
- net SBUS_5V_SEL*: now also U3.31 (2B10); no longer U3.3 (1A2)
- net SBUS_5V_SIZ[0]: now also U2.42 (1B12); no longer U2.15 (2A1)
- net SBUS_5V_SIZ[1]: now also U2.41 (2B1); no longer U2.16 (2A2)
- net SBUS_5V_SIZ[2]: now also U2.44 (1B10); no longer U2.18 (2A3)
- net SBUS_OE: now also U10.1 (~OE), U4.1 (~OE)
- no-connect marks 0 -> 1
Other:
- note removed: "BEWARE\nthe order\n(for routing)"
- note removed: "BR, BG: Master only\n(one-way each, of opposite direction)\nDP: not really used"
- note removed: "Inputs only"
- note removed: "outputs only\n(inputs on master)"
- moved on the sheet: C13, R13

Commit message: more V1.3
Parts:
- removed C7: 100nF 0402, Capacitor_SMD:C_0402_1005Metric, symbol Device:C
- removed R5, R6: 10k, Resistor_SMD:R_0402_1005Metric, symbol Device:R
- removed U_INT3: 74LVC2G07, For_SeeedStudio:SOT65P210X110-6N, symbol 74xGxx:74AUC2G07
- SBus1: DNP (none) -> DNP
Connections:
- net SBUS_3V3_INT[1]* is gone; now on net SBUS_3V3_INT[2]*: R2.2, U_INT2.3
- net SBUS_3V3_INT[2]*: no longer R1.2, U_INT2.1
- net SBUS_3V3_INT[3]*: now also R1.2, U_INT2.1; no longer R31.2, U_INT1.3
- net SBUS_3V3_INT[4]*: now also R31.2, U_INT1.3; no longer R30.2, U_INT1.1
- net SBUS_3V3_INT[5]*: now also R30.2, U_INT1.1
- net SBUS_5V_INT[1]*: no longer U_INT2.4
- net SBUS_5V_INT[2]*: now also U_INT2.4; no longer U_INT2.6
- net SBUS_5V_INT[3]*: now also U_INT2.6; no longer U_INT1.4
- net SBUS_5V_INT[4]*: now also U_INT1.4; no longer U_INT1.6
- net SBUS_5V_INT[5]*: now also U_INT1.6
