File: sbus-to-ztex/sbus-to-ztex.kicad_pcb (KiCad board)
At the start: 4 copper layers, 99.7 x 83.8 mm, 67 parts, among them J2 10118194-0001LF (USB micro-B), J3 Conn_02x07_Odd_Even, J4 10029449-111RLF (HDMI A), J6 Conn_01x03_Male, P1 DM3CS-SF, U1 SN74CB3T16211DGGR, U10 74CB3T1G125, U2 SN74CB3T16211DGGR, U3 SN74CB3T16211DGGR, U4 74CB3T1G125, U5 TPS2051CDBV, U6 SRV05-4, U7 TPD12S016PWR, U8 PCT2075DP, U9 PCT2075DP, X1 ASE-xxxMHz

Commit message: more V1.3
Parts:
- removed C23: 10nF 0402, Capacitor_SMD:C_0402_1005Metric
- removed C7: 100nF 0402, Capacitor_SMD:C_0402_1005Metric
- removed P1: DM3CS-SF, For_SeeedStudio:HRS_DM3CS-SF
- removed R5, R6: 10k, Resistor_SMD:R_0402_1005Metric
- removed U9: PCT2075DP, For_SeeedStudio:TSSOP-8_3x3mm_P0.65mm_ForSeeedStudio
- removed U_INT3: 74LVC2G07, For_SeeedStudio:SOT65P210X110-6N
- added GRAPHIC1: LogoLitex, For_SeeedStudio:litex_logo, F.Cu at (139.5, 72.8)
- added GRAPHIC2: LogoNetBSD, For_SeeedStudio:netbsd_logo, F.Cu at (138.4, 103.7)
- added J1: A2541HWR-2x6P (Pmod 2x6 F R), Connector_PinSocket_2.54mm:PinSocket_2x06_P2.54mm_Horizontal, F.Cu at (109.5, 65.0)
- added J5: Conn_01x04_Male, Connector_JST:JST_SH_BM04B-SRSS-TB_1x04-1MP_P1.00mm_Vertical, F.Cu at (166.0, 130.8)
- C1: value 47uF 10V 1206 -> 100nF; footprint Capacitor_SMD:C_1206_3216Metric -> Capacitor_SMD:C_0402_1005Metric
- C2: value 100nF 0402 -> 100nF
- moved C2 88.4 mm to (167.0, 125.8), turned to 0 degrees
- moved C1 7.50 mm to (113.5, 65.0), turned to 0 degrees
- moved C25 5.05 mm to (114.1, 83.0), turned to 180 degrees
- moved C9 0.75 mm to (177.5, 55.5)
- moved J6 0.75 mm to (182.8, 52.0)
Connections:
- J2 pad : (no net) -> SHIELD
- JAB1 pad 11: SBUS_3V3_AS* -> SBUS_3V3_SEL*
- JAB1 pad 12: SBUS_3V3_SEL* -> SBUS_3V3_D[00]
- JAB1 pad 13: SBUS_3V3_D[01] -> SBUS_3V3_D[02]
- JAB1 pad 14: SBUS_3V3_D[02] -> SBUS_3V3_D[03]
- JAB1 pad 15: SBUS_3V3_D[04] -> SBUS_3V3_D[05]
- JAB1 pad 16: SBUS_3V3_D[05] -> SBUS_3V3_D[06]
- JAB1 pad 17: SBUS_3V3_D[07] -> SBUS_3V3_D[08]
- JAB1 pad 18: SBUS_3V3_D[08] -> SBUS_3V3_D[09]
- JAB1 pad 19: SBUS_3V3_D[10] -> SBUS_3V3_D[11]
- JAB1 pad 21: SBUS_3V3_D[12] -> SBUS_3V3_D[14]
- JAB1 pad 22: SBUS_3V3_D[13] -> SBUS_3V3_D[15]
- JAB1 pad 23: SBUS_3V3_D[15] -> SBUS_3V3_D[17]
- JAB1 pad 24: SBUS_3V3_D[16] -> SBUS_3V3_D[18]
- JAB1 pad 25: SBUS_3V3_D[18] -> SBUS_3V3_D[20]
- JAB1 pad 26: SBUS_3V3_D[19] -> SBUS_3V3_D[21]
- JAB1 pad 27: SBUS_3V3_D[21] -> SBUS_3V3_D[23]
- JAB1 pad 28: SBUS_3V3_D[22] -> SBUS_3V3_D[24]
- JAB1 pad 9: SBUS_3V3_INT[1]* -> SBUS_3V3_AS*
- JCD1 pad 15: SBUS_3V3_INT[6]* -> SBUS_3V3_D[01]
- JCD1 pad 17: SBUS_3V3_D[00] -> SBUS_3V3_D[04]
- JCD1 pad 19: SBUS_3V3_D[03] -> SBUS_3V3_D[07]
- JCD1 pad 21: SBUS_3V3_D[06] -> SBUS_3V3_D[10]
- JCD1 pad 23: SBUS_3V3_D[09] -> SBUS_3V3_D[12]
- JCD1 pad 24: SBUS_3V3_D[11] -> SBUS_3V3_D[13]
- JCD1 pad 25: SBUS_3V3_D[14] -> SBUS_3V3_D[16]
- JCD1 pad 26: SBUS_3V3_D[17] -> SBUS_3V3_D[19]
- JCD1 pad 27: SBUS_3V3_D[20] -> SBUS_3V3_D[22]
- JCD1 pad 28: SBUS_3V3_D[23] -> SBUS_3V3_D[25]
- JCD1 pad 29: SBUS_3V3_D[24] -> SBUS_3V3_D[26]
- JCD1 pad 30: SBUS_3V3_D[25] -> SBUS_3V3_D[27]
- JCD1 pad 37: SBUS_3V3_D[27] -> SBUS_3V3_D[28]
- JCD1 pad 38: SBUS_3V3_D[26] -> SBUS_3V3_D[29]
- JCD1 pad 39: SBUS_3V3_D[28] -> SBUS_3V3_SIZ[1]
- JCD1 pad 41: SBUS_3V3_D[29] -> SBUS_3V3_SIZ[2]
- JCD1 pad 42: SD_D2 -> PMOD-1112+
- JCD1 pad 43: SBUS_3V3_SIZ[1] -> SBUS_3V3_PA[03]
- JCD1 pad 44: SD_D3 -> PMOD-1112-
- JCD1 pad 45: SBUS_3V3_SIZ[2] -> SBUS_3V3_PA[04]
- JCD1 pad 46: SD_CMD -> PMOD-910-
- JCD1 pad 47: SBUS_3V3_PA[03] -> SBUS_3V3_PA[06]
- JCD1 pad 48: SD_CLK -> PMOD-910+
- JCD1 pad 49: SBUS_3V3_PA[04] -> SBUS_3V3_PA[11]
- JCD1 pad 50: SD_D0 -> PMOD-78-
- JCD1 pad 51: SBUS_3V3_PA[06] -> SBUS_3V3_PA[13]
- JCD1 pad 52: SD_D1 -> PMOD-78+
- JCD1 pad 53: SBUS_3V3_PA[11] -> SBUS_3V3_PA[14]
- JCD1 pad 54: SBUS_3V3_PA[13] -> PMOD-56+
- JCD1 pad 55: SBUS_3V3_PA[14] -> SBUS_3V3_ACK[1]*
- JCD1 pad 56: SBUS_3V3_ACK[1]* -> PMOD-56-
- R1 pad 2: SBUS_3V3_INT[2]* -> SBUS_3V3_INT[3]*
- R2 pad 2: SBUS_3V3_INT[1]* -> SBUS_3V3_INT[2]*
- R30 pad 2: SBUS_3V3_INT[4]* -> SBUS_3V3_INT[5]*
- R31 pad 2: SBUS_3V3_INT[3]* -> SBUS_3V3_INT[4]*
- SBus1 pad 04: SBUS_5V_INT[1]* -> (no net)
- SBus1 pad 24: SBUS_5V_INT[6]* -> (no net)
- U_INT1 pad 1: SBUS_3V3_INT[4]* -> SBUS_3V3_INT[5]*
- U_INT1 pad 3: SBUS_3V3_INT[3]* -> SBUS_3V3_INT[4]*
- U_INT1 pad 4: SBUS_5V_INT[3]* -> SBUS_5V_INT[4]*
- U_INT1 pad 6: SBUS_5V_INT[4]* -> SBUS_5V_INT[5]*
- U_INT2 pad 1: SBUS_3V3_INT[2]* -> SBUS_3V3_INT[3]*
- U_INT2 pad 3: SBUS_3V3_INT[1]* -> SBUS_3V3_INT[2]*
- U_INT2 pad 4: SBUS_5V_INT[1]* -> SBUS_5V_INT[2]*
- U_INT2 pad 6: SBUS_5V_INT[2]* -> SBUS_5V_INT[3]*
Routing:
- net SBUS_3V3_INT[6]*: track 70.8 -> 0.00 mm, vias 1 -> 0
- net SBUS_3V3_D[17]: track 51.7 -> 15.5 mm
- net SBUS_3V3_D[11]: track 52.3 -> 16.2 mm
- net SBUS_3V3_D[23]: track 51.7 -> 17.4 mm
- net SBUS_3V3_D[13]: track 18.9 -> 52.7 mm
- net SBUS_3V3_D[07]: track 16.6 -> 50.3 mm
- net SBUS_3V3_D[10]: track 16.0 -> 49.7 mm
- net SBUS_3V3_D[04]: track 16.4 -> 50.1 mm
- net SBUS_3V3_D[01]: track 16.9 -> 50.6 mm
- net SBUS_3V3_D[12]: track 15.6 -> 49.3 mm
- net SBUS_3V3_D[14]: track 49.1 -> 15.8 mm
- net SBUS_3V3_D[20]: track 48.7 -> 15.9 mm
- net SBUS_3V3_D[19]: track 19.5 -> 51.3 mm
- net SBUS_3V3_D[09]: track 50.5 -> 19.4 mm
- net SBUS_3V3_D[03]: track 51.0 -> 19.8 mm
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Other:
- outline, holes or cut-outs redrawn
- board text added: "+3V3"
- board text added: "Fan 5V *low power*"
- board text added: "GND"
- board text added: "SCL"
- board text added: "SDA"
- board text added: "qwiic"

Commit message: logo
Parts:
- moved GRAPHIC2 7.91 mm to (144.6, 108.6)
- moved C9 3.00 mm to (174.5, 55.5)
- moved J6 3.00 mm to (179.8, 52.0)
- moved GRAPHIC1 0.15 mm to (139.5, 72.9)
Routing:
- net +5V: track 95.1 -> 97.0 mm
- net GND: track 104.7 -> 106.3 mm, vias 51 -> 76
