File: sbus-to-ztex/sbus-to-ztex.kicad_pcb (KiCad board)
At the start: 4 copper layers, 99.7 x 83.8 mm, 64 parts, among them J1 A2541HWR-2x6P (Pmod 2x6 F R), J2 10118194-0001LF (USB micro-B), J3 Conn_02x07_Odd_Even, J4 10029449-111RLF (HDMI A), J5 Conn_01x04_Male, J6 Conn_01x03_Male, U1 SN74CB3T16211DGGR, U10 74CB3T1G125, U2 SN74CB3T16211DGGR, U3 SN74CB3T16211DGGR, U4 74CB3T1G125, U5 TPS2051CDBV, U6 SRV05-4, U7 TPD12S016PWR, U8 PCT2075DP, X1 ASE-xxxMHz

Commit message: minor upd
Routing:
- net +5V: track 97.0 -> 99.6 mm

Commit message: details
Connections:
- J2 pad : SHIELD -> (no net)
Routing:
- net +5V: track 99.6 -> 102.6 mm
- net GND: vias 76 -> 56
Other:
- board text added: "USB"
- board text added: "pmod"
Changed lines of the file:
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@@
   (general
     (thickness 1.6)
-    (drawings 57)
-    (tracks 2723)
+    (drawings 59)
+    (tracks 2705)
     (zones 0)
     (modules 64)
@@
     (pad 6 smd rect (at -2.9 1.3 270) (size 1.2 1.55) (layers F.Cu F.Paste F.Mask)
       (net 98 SHIELD))
-    (pad "" smd oval (at 3.5 1.3 270) (size 0.89 1.55) (layers F.Paste)
-      (net 98 SHIELD))
+    (pad "" smd oval (at 3.5 1.3 270) (size 0.89 1.55) (layers F.Paste))
     (pad 6 smd rect (at 1 1.3 270) (size 1.5 1.55) (layers F.Cu F.Paste F.Mask)
       (net 98 SHIELD))
@@
     (pad 6 thru_hole oval (at 2.5 -1.4 270) (size 1.25 0.95) (drill oval 0.85 0.55) (layers *.Cu *.Mask)
       (net 98 SHIELD))
-    (pad "" smd oval (at -3.5 1.3 270) (size 0.89 1.55) (layers F.Paste)
-      (net 98 SHIELD))
+    (pad "" smd oval (at -3.5 1.3 270) (size 0.89 1.55) (layers F.Paste))
     (pad 6 thru_hole oval (at -2.5 -1.4 270) (size 1.25 0.95) (drill oval 0.85 0.55) (layers *.Cu *.Mask)
       (net 98 SHIELD))
@@
     )
   )
+  (gr_text USB (at 99.4 121.4) (layer F.SilkS)
+    (effects (font (size 1 1) (thickness 0.15) italic))
+  )
+  (gr_text pmod (at 103.4 80.2) (layer F.SilkS)
+    (effects (font (size 1 1) (thickness 0.15) italic))
+  )
   (gr_text 1 (at 113.39 88.04) (layer F.SilkS)
     (effects (font (size 0.75 0.75) (thickness 0.15)))
   )
   (gr_circle (center 110 131) (end 111.6 131) (layer Edge.Cuts) (width 0.15))
-  (gr_text "Fan\n5V *low power*" (at 174.13 58.85) (layer F.SilkS)
-    (effects (font (size 1 1) (thickness 0.2)))
+  (gr_text "Fan\n5V *low power*" (at 174.6 58.85) (layer F.SilkS)
+    (effects (font (size 1 1) (thickness 0.2) italic))
   )
   (gr_text qwiic (at 162.31 127.43) (layer F.SilkS)
-    (effects (font (size 1 1) (thickness 0.15)))
+    (effects (font (size 1 1) (thickness 0.15) italic))
   )
   (gr_text SCL (at 164.41 126.04 90) (layer F.SilkS)
@@
   )
   (gr_text JTAG (at 147.29 54.71 90) (layer F.SilkS)
-    (effects (font (size 1 1) (thickness 0.15)))
+    (effects (font (size 1 1) (thickness 0.15) italic))
   )
   (gr_text 1 (at 116.98 103.95) (layer F.SilkS)
@@
   )
   (gr_circle (center 110 118) (end 111.6 118) (layer Edge.Cuts) (width 0.15))
-  (gr_text "ZTex 2.13 outline\n" (at 162.08 93.4 -90) (layer F.SilkS)
-    (effects (font (size 1.5 1.5) (thickness 0.3)))
+  (gr_text "ZTex 2.13 outline\n" (at 166.8 57.6 -90) (layer F.SilkS)
+    (effects (font (size 1 1) (thickness 0.2)))
   )
   (gr_line (start 168.45 133.82) (end 117.65 133.82) (layer F.SilkS) (width 0.2))
@@
   (gr_line (start 97 50) (end 196.7 50) (layer Edge.Cuts) (width 0.15))
   (segment (start 188.289678 117.295) (end 186.634678 118.95) (width 0.1524) (layer B.Cu) (net 0))
-  (via (at 138.605 57.64) (size 0.8) (drill 0.4) (layers F.Cu B.Cu) (net 1))
   (via (at 177.25 110.25) (size 0.8) (drill 0.4) (layers F.Cu B.Cu) (net 1))
   (via (at 172.75 110.25) (size 0.8) (drill 0.4) (layers F.Cu B.Cu) (net 1))
@@
   (via (at 112.25 83.04) (size 0.8) (drill 0.4) (layers F.Cu B.Cu) (net 1))
   (segment (start 113.615 83.04) (end 112.25 83.04) (width 0.25) (layer F.Cu) (net 1))
-  (via (at 138.605 60.18) (size 0.8) (drill 0.4) (layers F.Cu B.Cu) (net 1))
-  (via (at 138.605 62.72) (size 0.8) (drill 0.4) (layers F.Cu B.Cu) (net 1))
-  (via (at 138.605 65.26) (size 0.8) (drill 0.4) (layers F.Cu B.Cu) (net 1))
-  (via (at 138.605 67.8) (size 0.8) (drill 0.4) (layers F.Cu B.Cu) (net 1))
-  (via (at 138.605 70.34) (size 0.8) (drill 0.4) (layers F.Cu B.Cu) (net 1))
-  (via (at 138.605 72.88) (size 0.8) (drill 0.4) (layers F.Cu B.Cu) (net 1))
-  (via (at 138.605 75.42) (size 0.8) (drill 0.4) (layers F.Cu B.Cu) (net 1))
-  (via (at 138.605 77.96) (size 0.8) (drill 0.4) (layers F.Cu B.Cu) (net 1))
-  (via (at 138.605 80.5) (size 0.8) (drill 0.4) (layers F.Cu B.Cu) (net 1))
-  (via (at 138.605 83.04) (size 0.8) (drill 0.4) (layers F.Cu B.Cu) (net 1))
-  (via (at 138.605 85.58) (size 0.8) (drill 0.4) (layers F.Cu B.Cu) (net 1))
-  (via (at 138.605 88.12) (size 0.8) (drill 0.4) (layers F.Cu B.Cu) (net 1))
-  (via (at 138.605 90.66) (size 0.8) (drill 0.4) (layers F.Cu B.Cu) (net 1))
-  (via (at 138.605 93.2) (size 0.8) (drill 0.4) (layers F.Cu B.Cu) (net 1))
-  (via (at 138.605 95.74) (size 0.8) (drill 0.4) (layers F.Cu B.Cu) (net 1))
-  (via (at 138.605 98.28) (size 0.8) (drill 0.4) (layers F.Cu B.Cu) (net 1))
-  (via (at 138.605 100.82) (size 0.8) (drill 0.4) (layers F.Cu B.Cu) (net 1))
-  (via (at 138.605 103.36) (size 0.8) (drill 0.4) (layers F.Cu B.Cu) (net 1))
-  (via (at 138.605 105.9) (size 0.8) (drill 0.4) (layers F.Cu B.Cu) (net 1))
-  (via (at 138.605 108.44) (size 0.8) (drill 0.4) (layers F.Cu B.Cu) (net 1))
-  (via (at 138.605 110.98) (size 0.8) (drill 0.4) (layers F.Cu B.Cu) (net 1))
-  (via (at 138.605 113.52) (size 0.8) (drill 0.4) (layers F.Cu B.Cu) (net 1))
-  (via (at 138.605 116.06) (size 0.8) (drill 0.4) (layers F.Cu B.Cu) (net 1))
   (segment (start 109.63 101) (end 110.665 101) (width 0.25) (layer F.Cu) (net 1))
   (via (at 111.1 101.435) (size 0.45) (drill 0.3) (layers F.Cu B.Cu) (net 1))
   (segment (start 110.665 101) (end 111.1 101.435) (width 0.25) (layer F.Cu) (net 1))
+  (via (at 182.5 78) (size 0.8) (drill 0.4) (layers F.Cu B.Cu) (net 1))
+  (via (at 162.5 78) (size 0.8) (drill 0.4) (layers F.Cu B.Cu) (net 1))
+  (via (at 162.5 98) (size 0.8) (drill 0.4) (layers F.Cu B.Cu) (net 1))
+  (via (at 162.5 118) (size 0.8) (drill 0.4) (layers F.Cu B.Cu) (net 1))
   (segment (start 153.21 131.3) (end 155.75 131.3) (width 1) (layer In2.Cu) (net 2))
   (segment (start 153.21 131.3) (end 150 131.3) (width 1) (layer In2.Cu) (net 2))
@@
   (segment (start 179.75 54.54) (end 177.79 54.54) (width 1) (layer In2.Cu) (net 2))
   (segment (start 155.75 131.3) (end 153.21 131.3) (width 1) (layer F.Cu) (net 2))
+  (segment (start 153.21 131.3) (end 153.21 132.81) (width 1) (layer In2.Cu) (net 2))
+  (segment (start 155.75 131.3) (end 155.75 132.85) (width 1) (layer In2.Cu) (net 2))
   (via (at 178.75 118.95) (size 0.45) (drill 0.3) (layers F.Cu B.Cu) (net 3))
   (segment (start 178.45 118.65) (end 178.75 118.95) (width 0.1524) (layer F.Cu) (net 3))
@@
     )
   )
-  (zone (net 9) (net_name +3V3) (layer In2.Cu) (hatch edge 0.508)
+  (zone (net 2) (net_name +5V) (layer In2.Cu) (hatch edge 0.508)
     (connect_pads (clearance 0.254))
     (min_thickness 0.254)
-    (fill yes (arc_segments 32) (thermal_gap 0.254) (thermal_bridge_width 0.508) (smoothing fillet) (radius 0.25))
+    (fill yes (arc_segments 32) (thermal_gap 0.508) (thermal_bridge_width 0.508) (smoothing fillet) (radius 0.25))
     (polygon
       (pts
-        (xy 181.75 59.75) (xy 181.75 129.5) (xy 97 129.5) (xy 97 50) (xy 176.75 50)
-        (xy 176.75 59.75)
+        (xy 196.5 133.5) (xy 114.75 133.5) (xy 114.75 130) (xy 182.25 130) (xy 182.25 59.25)
+        (xy 177.25 59.25) (xy 177.25 50) (xy 196.5 50)
       )
     )
   )
-  (zone (net 2) (net_name +5V) (layer In2.Cu) (hatch edge 0.508)
+  (zone (net 9) (net_name +3V3) (layer In2.Cu) (hatch edge 0.508)
     (connect_pads (clearance 0.254))
     (min_thickness 0.254)
-    (fill yes (arc_segments 32) (thermal_gap 0.508) (thermal_bridge_width 0.508) (smoothing fillet) (radius 0.25))
+    (fill yes (arc_segments 32) (thermal_gap 0.254) (thermal_bridge_width 0.508) (smoothing fillet) (radius 0.25))
     (polygon
       (pts
-        (xy 196.5 133.5) (xy 114.75 133.5) (xy 114.75 130) (xy 182.25 130) (xy 182.25 59.25)
-        (xy 177.25 59.25) (xy 177.25 50) (xy 196.5 50)
+        (xy 181.75 59.75) (xy 181.75 129.5) (xy 97 129.5) (xy 97 50) (xy 176.75 50)
+        (xy 176.75 59.75)
       )
     )
