File: sbus-to-ztex/pmod.sch (KiCad schematic (older format))
At the start: 2 parts, among them J1 A2541HWR-2x6P (Pmod 2x6 F R)

Commit message: details
Other:
- note removed: "Dual-row "extended" Pmod\nExternal, in line w/ the carrier"
Changed lines of the file:
@@
 Comment4 ""
 $EndDescr
-Text Notes 7300 2850 0    50   ~ 0
-Dual-row "extended" Pmod\nExternal, in line w/ the carrier
 Text GLabel 7150 3500 0    50   Input ~ 0
 PMOD-56-
